File: kicad/pipico_vga.kicad_sch (KiCad schematic)
At the start: 66 parts, among them J1 RJ45_LED_Shielded, J2 DB15_Male_HighDensity_Mountin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, J3 power, Q1 2N7002P, Q2 2N7002P, Q3 CPH3350-TL-W, U1 Pico, U2 74LVC162244ADGVJ, U3 AP62250

Commit message: Rev 4 of main board
controller rev1 done as well :D
Parts:
- removed Q1, Q2: 2N7002P, Package_TO_SOT_SMD:SOT-23_Handsoldering, symbol Device:Q_NMOS_GSD
- added C10, C9: 4u7, Capacitor_SMD:C_0603_1608Metric_Pad1.08x0.95mm_HandSolder, symbol Device:C_Small
- added C11: 100n, Capacitor_SMD:C_0603_1608Metric_Pad1.08x0.95mm_HandSolder, symbol Device:C
- added H5: MountingHole_Pad, MountingHole:MountingHole_3.2mm_M3_DIN965_Pad, symbol Mechanical:MountingHole_Pad
- added J4: RJE37-188-2410, Connector_RJ:RJ45_Amphenol_RJHSE538X, symbol Connector:RJ45_LED_Shielded
- added R33, R34: 10k, Resistor_SMD:R_0603_1608Metric_Pad0.98x0.95mm_HandSolder, symbol Device:R_Small
- added R35, R36: 1k, Resistor_SMD:R_0603_1608Metric_Pad0.98x0.95mm_HandSolder, symbol Device:R_Small
- added U4: PI3C3305LE, Package_SO:TSSOP-8_4.4x3mm_P0.65mm, symbol good_things:PI3C3305LE
- C1, C2, C3, C4, C6, C7, C8: footprint Capacitor_SMD:C_0603_1608Metric_Pad1.05x0.95mm_HandSolder -> Capacitor_SMD:C_0603_1608Metric_Pad1.08x0.95mm_HandSolder
- J1: value RJ45_LED_Shielded -> RJE37-188-2410; footprint Connector_RJ:RJ45_BEL_SS74301-00x_Vertical -> Connector_RJ:RJ45_Amphenol_RJHSE538X
- R1, R10, R11, R12, R13, R14, R15, R16, R17, R18, R19, R2, R20, R21, R22, R23, R24, R25, R26, R27, R28, R29, R3, R30, R31, R32, R4, R5, R6, R7, R8, R9: footprint Resistor_SMD:R_0603_1608Metric_Pad1.05x0.95mm_HandSolder -> Resistor_SMD:R_0603_1608Metric_Pad0.98x0.95mm_HandSolder
Connections:
- net led0 is gone; now on net connected_0_n: U1.29 (GPIO22)
- net +3V3: now also J1.8, R28.1, R29.1, C10.1, C11.1, C9.1, J4.8, R33.1, R34.1, R36.1, U4.8 (VCC); no longer J1.10, J1.12, J1.3
- net +5V: now also R35.1
- net GND: now also J1.7, J1.9, C10.2, C11.2, C9.2, H5.1, J4.11, J4.7, J4.SH, U4.4 (GND); no longer J1.8
- net vga_clk: now also U1.32 (GPIO27_ADC1); no longer U1.25 (GPIO19)
- net vga_data: now also U1.31 (GPIO26_ADC0); no longer U1.24 (GPIO18)
- net ie_n: now reaches U1.34 (GPIO28_ADC2)
- net ie_n: now also J1.4, J4.4
- net connected_0_n: now reaches J1.11
- net connected_0_n: now also J1.5, R33.2, U4.1 (BE1); no longer R28.1
- net copi: now reaches J1.6
- net copi: now also U1.25 (GPIO19), U4.2 (A1)
- net at R28.2: now also J1.12
- net at R29.2: now also J4.10
- net connected: no longer names the net of U1.26 (GPIO20)
- net connected: no longer J1.7
- net led1 renamed connected_1_n
- net connected_1_n: now also J4.5, J4.9, R34.2, U4.7 (BE2)
- net rx renamed clk
- net clk: now also U1.24 (GPIO18), J4.2; no longer U1.22 (GPIO17)
- net tx renamed cipo
- net cipo: now also J4.1, U4.6 (B2); no longer J1.1
- new net: J4.12, R36.2
- new net: J1.10, R35.2
- new net dshift: J1.1, J4.6, U4.3 (B1), U4.5 (A2)
- new net out_shift_clk: J1.3, J4.3, U1.22 (GPIO17)
- no-connect marks 11 -> 17
Other:
- note added: "Bypasses controller in shift register chain if the controller is not connected"
- note added: "SPI0 19: TX (COPI) 18: clk 17: CSn 16 RX (CIPO)"
- note added: "uses i2c1"
- moved on the sheet: C1, C2, C3, C4, C5, C6, C7, C8, D1, F1, GND1, GND2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

Commit message: Half working sw
Other:
- note added: "resistor values for dac with 75 ohm term solve: 0.7/2^i=3.3*75/(75+x) i=1: 632.1 i=2: 1339 i=3: 2753 i=4: 5582"
Changed lines of the file:
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@@
+    (effects (font (size 1.27 1.27)) (justify left bottom))
+  )
+  (text "resistor values for dac with 75 ohm term\nsolve: 0.7/2^i=3.3*75/(75+x)\ni=1: 632.1\ni=2: 1339\ni=3: 2753\ni=4: 5582"
+    (at 111.76 40.005 0)
     (effects (font (size 1.27 1.27)) (justify left bottom))
   )
